File: Single_transistor_AMP.sch (KiCad schematic (older format))
At the start: 10 parts, among them J1 9V_IN, J2 SIG_OUT, J3 SIG_IN, Q1 BC547

Commit message: Set design rules, created PCB layout and traces, positioned labels
Connections:
- net GND: now reaches C2.1, J1.1 (Pin_1), J3.1 (Pin_1), R3.2, R4.2
- net GND: now also J2.1 (Pin_1); no longer J2.2 (Pin_2)
- net at Q1.3 (C), R1.2: now also J2.2 (Pin_2); no longer J2.1 (Pin_1)
Changed lines of the file:
@@
 L Connector:Screw_Terminal_01x02 J2
 U 1 1 5E71D6F3
-P 4400 2950
-F 0 "J2" H 4479 2942 50  0000 L CNN
-F 1 "SIG_OUT" H 4479 2851 50  0000 L CNN
-F 2 "TerminalBlock:TerminalBlock_bornier-2_P5.08mm" H 4400 2950 50  0001 C CNN
-F 3 "~" H 4400 2950 50  0001 C CNN
-	1    4400 2950
-	1    0    0    -1
+P 4400 3050
+F 0 "J2" H 4479 3042 50  0000 L CNN
+F 1 "SIG_OUT" H 4479 2951 50  0000 L CNN
+F 2 "TerminalBlock:TerminalBlock_bornier-2_P5.08mm" H 4400 3050 50  0001 C CNN
+F 3 "~" H 4400 3050 50  0001 C CNN
+	1    4400 3050
+	1    0    0    1
 $EndComp
 Wire Wire Line
 	3550 2950 4200 2950
 Wire Wire Line
-	4200 3050 4200 3700
+	4200 3050 4200 3200
 Wire Wire Line
 	4200 3700 3900 3700
@@
 	2550 2700 2500 2700
 Connection ~ 2550 3250
+$Comp
+L power:GND #PWR0101
+U 1 1 5E985070
+P 4200 3700
+F 0 "#PWR0101" H 4200 3450 50  0001 C CNN
+F 1 "GND" H 4205 3527 50  0000 C CNN
+F 2 "" H 4200 3700 50  0001 C CNN
+F 3 "" H 4200 3700 50  0001 C CNN
+	1    4200 3700
+	1    0    0    -1
+$EndComp
+Connection ~ 4200 3700
+$Comp
+L power:PWR_FLAG #FLG0101
+U 1 1 5E9853F6
+P 4200 3200
+F 0 "#FLG0101" H 4200 3275 50  0001 C CNN
+F 1 "PWR_FLAG" V 4200 3328 50  0000 L CNN
+F 2 "" H 4200 3200 50  0001 C CNN
+F 3 "~" H 4200 3200 50  0001 C CNN
+	1    4200 3200
+	0    1    1    0
+$EndComp
+Connection ~ 4200 3200
+Wire Wire Line
+	4200 3200 4200 3700
 $EndSCHEMATC
